File: kicad/ESC_v2/ESC_v2.kicad_pcb (KiCad board)
At the start: 2 copper layers, 50 x 50 mm, 141 parts, among them J1 Conn_01x05_Pin, J10 Conn_01x01_Pin, J11 Conn_01x01_Pin, J12 Conn_01x01_Pin, J13 Conn_01x03_Pin, J14 Conn_01x01_Pin, J15 Conn_01x01_Pin, J16 Conn_01x01_Pin, J2 Conn_01x05_Pin, J3 Conn_01x03_Pin, J4 Conn_01x03_Pin, J6 Conn_01x06_Pin, J7 Conn_01x02_Pin, J8 Conn_01x04_Pin, J9 Conn_01x02_Pin, Q1 RH6L040BGTB1, Q10 RH6L040BGTB1, Q11 RH6L040BGTB1, Q12 RH6L040BGTB1, Q2 RH6L040BGTB1, Q3 RH6L040BGTB1, Q4 RH6L040BGTB1, Q5 RH6L040BGTB1, Q6 RH6L040BGTB1, Q7 RH6L040BGTB1, Q8 RH6L040BGTB1, Q9 RH6L040BGTB1, U1 L6387, U10 BD4104, U11 AMS1117-5.0, U12 ACS711xEXLT-15AB, U13 LM2937xMP, U19 STM32G431CBUx, U2 L6387, U3 L6387, U4 L6387, U5 L6387, U6 L6387, U7 AMS1117-3.3, U8 ACS711xEXLT-15AB, U9 ACS711xEXLT-15AB

Commit message: a
Parts:
- J10, J11, J12, J14, J15, J16: moved to B.Cu
- moved C7 150.3 mm to (68.3, 87.6), turned to -90 degrees
- moved C8 145.5 mm to (68.5, 92.9), turned to -90 degrees
- moved C14 144.5 mm to (68.4, 98.4), turned to -90 degrees
- moved C4 138.5 mm to (68.0, 54.1), turned to -90 degrees
- moved C13 135.6 mm to (68.0, 59.5), turned to -90 degrees
- moved J9 134.4 mm to (86.3, 77.6), turned to -90 degrees
- moved C10 133.3 mm to (69.4, 92.9), turned to -90 degrees
- moved R40 132.6 mm to (98.3, 94.6)
- moved D8 132.2 mm to (97.1, 98.2), turned to -90 degrees
- moved D1 131.9 mm to (99.0, 97.0), turned to 90 degrees
- moved R56 130.2 mm to (35.1, 60.8)
- moved R57 130.2 mm to (35.1, 63.3)
- moved R58 130.2 mm to (35.1, 65.8)
- moved R59 130.2 mm to (35.1, 68.3)
- moved C16 129.9 mm to (74.9, 71.1)
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Routing:
- net VCC: track 0.00 -> 54.9 mm
- net OPAMP1_VINM0: track 0.00 -> 47.5 mm, vias 0 -> 7
- net +12V: track 0.00 -> 21.6 mm
- net VREF: track 0.00 -> 12.3 mm
- net +5V: track 0.00 -> 6.30 mm

Commit message: add ESC_v3 final ver
Parts:
- removed C31: 470u, Capacitor_SMD:C_Elec_10x10.2
- removed D1, D11, D4, D6, D9: BLUE, LED_SMD:LED_0805_2012Metric
- removed D10, D12, D3, D5, D7, D8: RED, LED_SMD:LED_0805_2012Metric
- removed J10, J11, J12, J14, J15, J16: Conn_01x01_Pin, TestPoint:TestPoint_Pad_3.0x3.0mm
- removed J13: Conn_01x03_Pin, Connector_Molex:Molex_KK-254_AE-6410-03A_1x03_P2.54mm_Vertical
- removed J4: Conn_01x03_Pin, Connector_PinSocket_2.54mm:PinSocket_1x03_P2.54mm_Vertical
- removed R37, R38, R39, R40, R41, R42: 4.7k, Resistor_SMD:R_0402_1005Metric_Pad0.72x0.64mm_HandSolder
- added C23: 0.1u, Capacitor_SMD:C_0402_1005Metric, F.Cu at (57.9, 81.6)
- added C39: 0.1u, Capacitor_SMD:C_0402_1005Metric, F.Cu at (57.2, 83.3)
- added C40: 22uF, Capacitor_SMD:C_0603_1608Metric, F.Cu at (79.6, 81.5)
- added C41: 22uF, Capacitor_SMD:C_0603_1608Metric, F.Cu at (79.6, 79.0)
- added C42: 22uF, Capacitor_SMD:C_0603_1608Metric, F.Cu at (79.6, 76.5)
- added C43: 22uF, Capacitor_SMD:C_0603_1608Metric, F.Cu at (79.6, 74.0)
- added C44: 22uF, Capacitor_SMD:C_0603_1608Metric, F.Cu at (79.6, 71.5)
- added C45: 22uF, Capacitor_SMD:C_0603_1608Metric, F.Cu at (82.6, 71.5)
- added C46: 22uF, Capacitor_SMD:C_0603_1608Metric, F.Cu at (82.6, 74.0)
- added C47: 22uF, Capacitor_SMD:C_0603_1608Metric, F.Cu at (82.6, 76.5)
- added C48: 22uF, Capacitor_SMD:C_0603_1608Metric, F.Cu at (82.6, 79.0)
- added C49: 22uF, Capacitor_SMD:C_0603_1608Metric, F.Cu at (82.6, 81.5)
- added J5: Conn_01x02_Pin, Connector_PinHeader_2.54mm:PinHeader_1x02_P2.54mm_Vertical, B.Cu at (64.3, 89.7)
- added NRST1: SW_Push, jisaku:Aitendo_SW SMD 6x3.5, B.Cu at (59.3, 78.9)
- added R5: 10k, Resistor_SMD:R_0402_1005Metric_Pad0.72x0.64mm_HandSolder, F.Cu at (57.2, 84.3)
- added R6: 10k, Resistor_SMD:R_0402_1005Metric_Pad0.72x0.64mm_HandSolder, F.Cu at (57.3, 80.1)
- added TP1: TestPoint, TestPoint:TestPoint_Pad_D1.0mm, F.Cu at (68.5, 51.0)
- added TP10: TestPoint, TestPoint:TestPoint_Pad_D1.0mm, F.Cu at (69.0, 91.1)
- added TP11: TestPoint, TestPoint:TestPoint_Pad_D1.0mm, F.Cu at (69.0, 95.1)
- added TP12: TestPoint, TestPoint:TestPoint_Pad_D1.0mm, F.Cu at (69.0, 96.6)
- added TP2: TestPoint, TestPoint:TestPoint_Pad_D1.0mm, F.Cu at (67.6, 52.3)
- added TP3: TestPoint, TestPoint:TestPoint_Pad_D1.0mm, F.Cu at (66.8, 56.4)
- added TP4: TestPoint, TestPoint:TestPoint_Pad_D1.0mm, F.Cu at (68.5, 57.5)
- added TP5: TestPoint, TestPoint:TestPoint_Pad_D1.0mm, F.Cu at (67.8, 61.3)
- added TP6: TestPoint, TestPoint:TestPoint_Pad_D1.0mm, F.Cu at (68.5, 63.0)
- added TP7: TestPoint, TestPoint:TestPoint_Pad_D1.0mm, F.Cu at (69.1, 84.2)
- added TP8: TestPoint, TestPoint:TestPoint_Pad_D1.0mm, F.Cu at (69.1, 85.8)
- added TP9: TestPoint, TestPoint:TestPoint_Pad_D1.0mm, F.Cu at (69.0, 89.4)
- added button1: SW_Push, jisaku:Aitendo_SW SMD 6x3.5, B.Cu at (59.3, 83.3)
- C38: value 1u -> 0.1u
- D15, D16, D17: footprint LED_SMD:LED_0805_2012Metric -> LED_SMD:LED_0603_1608Metric
- D2: value BLUE -> 1N5819WS; footprint LED_SMD:LED_0805_2012Metric -> Diode_SMD:D_SOD-323
- J1, J2, J6, J8, R10, R19, R20, R28, R34, R4: moved to B.Cu
- J3: value Conn_01x03_Pin -> Conn_01x01_Pin; footprint Connector_PinSocket_2.54mm:PinSocket_1x03_P2.54mm_Vertical -> Connector_PinHeader_1.00mm:PinHeader_1x01_P1.00mm_Vertical
- J7: footprint Connector_JST:JST_XH_B2B-XH-AM_1x02_P2.50mm_Vertical -> Connector_JST:JST_XH_S2B-XH-A_1x02_P2.50mm_Horizontal; moved to B.Cu
- R48, R49, R54: value 22k -> 68k
- R51: footprint Resistor_SMD:R_0402_1005Metric_Pad0.72x0.64mm_HandSolder -> Resistor_SMD:R_2010_5025Metric_Pad1.40x2.65mm_HandSolder
- moved J7 114.0 mm to (59.7, 90.9), turned to 90 degrees
- moved D13 88.5 mm to (52.1, 76.3)
- moved D15 88.5 mm to (52.1, 78.9)
- moved D16 88.5 mm to (52.1, 81.5)
- moved D17 88.5 mm to (52.1, 84.0)
- moved R47 86.5 mm to (84.5, 66.4), turned to -90 degrees
- moved R46 84.8 mm to (84.5, 60.8), turned to -90 degrees
- moved R48 84.1 mm to (82.9, 67.0)
- moved J6 83.6 mm to (65.7, 58.0), turned to -90 degrees
- moved D14 81.6 mm to (54.0, 71.3)
- moved R53 81.3 mm to (82.9, 66.0), turned to 180 degrees
- moved R50 80.9 mm to (82.8, 60.3), turned to 180 degrees
- moved R49 80.0 mm to (82.8, 61.3)
- moved R52 78.3 mm to (84.5, 55.3), turned to -90 degrees
- moved R54 74.8 mm to (82.9, 55.9)
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Connections:
- net TIM4_CH1 renamed TIM4_CH2
- C1 pad 2: OPAMP1_VINM0 -> GND
- C10 pad 2: OPAMP1_VINM0 -> GND
- C13 pad 2: OPAMP1_VINM0 -> GND
- C14 pad 2: OPAMP1_VINM0 -> GND
- C15 pad 2: OPAMP1_VINM0 -> GND
- C16 pad 2: OPAMP1_VINM0 -> GND
- C17 pad 2: OPAMP1_VINM0 -> GND
- C19 pad 2: OPAMP1_VINM0 -> GND
- C20 pad 2: OPAMP1_VINM0 -> GND
- C21 pad 2: OPAMP1_VINM0 -> GND
- C25 pad 2: OPAMP1_VINM0 -> GND
- C26 pad 2: OPAMP1_VINM0 -> GND
- C27 pad 2: OPAMP1_VINM0 -> GND
- C28 pad 2: OPAMP1_VINM0 -> GND
- C29 pad 1: +12V -> +5V
- C29 pad 2: OPAMP1_VINM0 -> GND
- C3 pad 2: OPAMP1_VINM0 -> GND
- C30 pad 2: OPAMP1_VINM0 -> GND
- C32 pad 2: OPAMP1_VINM0 -> GND
- C33 pad 2: OPAMP1_VINM0 -> GND
- C34 pad 2: OPAMP1_VINM0 -> GND
- C35 pad 2: OPAMP1_VINM0 -> GND
- C36 pad 2: OPAMP1_VINM0 -> GND
- C37 pad 2: OPAMP1_VINM0 -> GND
- C38 pad 2: OPAMP1_VINM0 -> GND
- C4 pad 2: OPAMP1_VINM0 -> GND
- C5 pad 2: OPAMP1_VINM0 -> GND
- C7 pad 2: OPAMP1_VINM0 -> GND
- C8 pad 2: OPAMP1_VINM0 -> GND
- C9 pad 2: OPAMP1_VINM0 -> GND
- D13 pad 1: OPAMP1_VINM0 -> GND
- D14 pad 2: Net-(D14-DOUT) -> unconnected-(D14-DOUT-Pad2)
- D14 pad 3: OPAMP1_VINM0 -> GND
- D15 pad 1: OPAMP1_VINM0 -> GND
- D16 pad 1: OPAMP1_VINM0 -> GND
- D17 pad 1: OPAMP1_VINM0 -> GND
- D2 pad 1: /halfHbridge5/out1 -> +5V
- J1 pad 1: TIM3_CH1 -> +5V
- J1 pad 2: Net-(J1-Pin_2) -> TIM3_CH1
- J1 pad 4: TIM3_ETR -> TIM3_CH3
- J1 pad 5: OPAMP1_VINM0 -> GND
- J2 pad 1: TIM2_CH1 -> +5V
- J2 pad 2: Net-(J2-Pin_2) -> TIM2_CH1
- J2 pad 4: TIM2_ETR -> TIM2_CH3
- J2 pad 5: OPAMP1_VINM0 -> GND
- J3 pad 1: +5V -> GND
- J6 pad 1: unconnected-(J6-Pin_1-Pad1) -> +5V
- J6 pad 4: OPAMP1_VINM0 -> GND
- J7 pad 1: CAN_H -> CAN_L
- J7 pad 2: CAN_L -> CAN_H
- J8 pad 1: OPAMP1_VINM0 -> GND
- J9 pad 1: VCC -> GND
- J9 pad 2: OPAMP1_VINM0 -> VCC
- R43 pad 2: CAN_H -> Net-(J5-Pin_1)
- R44 pad 2: OPAMP1_VINM0 -> GND
- R45 pad 2: OPAMP1_VINM0 -> GND
- R50 pad 2: OPAMP1_VINM0 -> GND
- R51 pad 2: OPAMP1_VINM0 -> GND
- R53 pad 2: OPAMP1_VINM0 -> GND
- R55 pad 2: OPAMP1_VINM0 -> GND
- U1 pad 4: OPAMP1_VINM0 -> GND
- U10 pad 2: OPAMP1_VINM0 -> GND
- U10 pad 8: OPAMP1_VINM0 -> GND
- U11 pad 1: OPAMP1_VINM0 -> GND
- U11 pad 2: +5V -> Net-(D2-A)
- U12 pad 2: OPAMP1_VINM0 -> GND
- U12 pad 3: OPAMP1_VINM0 -> GND
- U13 pad 2: OPAMP1_VINM0 -> GND
- U19 pad 10: TX -> TIM2_CH3
- U19 pad 11: OPAMP1_VINM0 -> OPAMP1_VINP
- U19 pad 12: TIM3_CH2 -> ADC2_IN14
- U19 pad 13: OPAMP1_VINM0 -> ADC2_IN15
- U19 pad 14: TIM3_CH1 -> unconnected-(U19-PA6-Pad14)
- U19 pad 15: OPAMP1_VINP -> OPAMP2_VINP
- U19 pad 17: TIM1_CH2N -> TIM3_CH3
- U19 pad 18: TIM1_CH3N -> TIM8_CH3N
- U19 pad 19: OPAMP1_VINM0 -> OPAMP3_VINM0
- U19 pad 22: unconnected-(U19-PB10-Pad22) -> TX
- U19 pad 24: ADC2_IN14 -> RX
- U19 pad 27: OPAMP2_VINP -> TIM1_CH2N
- U19 pad 28: ADC2_IN15 -> TIM1_CH3N
- U19 pad 29: unconnected-(U19-PC6-Pad29) -> button
- U19 pad 38: TIM2_ETR -> TIM2_CH3
- U19 pad 41: TIM3_ETR -> TIM3_CH3
- U19 pad 42: RX -> TIM3_CH1
- U19 pad 43: TIM8_CH3N -> TIM3_CH2
- U19 pad 49: OPAMP1_VINM0 -> GND
- U19 pad 7: unconnected-(U19-PG10-Pad7) -> NRST
- U2 pad 4: OPAMP1_VINM0 -> GND
- U3 pad 4: OPAMP1_VINM0 -> GND
- U4 pad 4: OPAMP1_VINM0 -> GND
- U5 pad 4: OPAMP1_VINM0 -> GND
- U6 pad 4: OPAMP1_VINM0 -> GND
- U7 pad 1: OPAMP1_VINM0 -> GND
- U7 pad 3: +12V -> +5V
- U8 pad 2: OPAMP1_VINM0 -> GND
- U8 pad 3: OPAMP1_VINM0 -> GND
- U9 pad 2: OPAMP1_VINM0 -> GND
- U9 pad 3: OPAMP1_VINM0 -> GND
Routing:
- net GND: track 0.00 -> 360.4 mm, vias 0 -> 114
- net VREF: track 12.3 -> 193.3 mm, vias 0 -> 10
- net +5V: track 6.30 -> 113.9 mm, vias 0 -> 4
- net TIM2_CH3: track 0.00 -> 82.4 mm, vias 0 -> 3
- net ADC2_IN10: track 0.00 -> 72.1 mm, vias 0 -> 3
- net VCC: track 54.9 -> 126.9 mm, vias 0 -> 112
- net ADC2_IN14: track 0.00 -> 64.9 mm, vias 0 -> 5
- net ADC2_IN15: track 0.00 -> 64.7 mm, vias 0 -> 5
- net +12V: track 21.6 -> 81.7 mm, vias 0 -> 23
- net OPAMP1_VINP: track 0.00 -> 52.9 mm, vias 0 -> 3
- net OPAMP1_VINM0: track 47.5 -> 0.00 mm, vias 7 -> 0
- net TIM2_CH1: track 0.00 -> 46.2 mm, vias 0 -> 1
- net OPAMP2_VINP: track 0.00 -> 45.6 mm, vias 0 -> 3
- net NRST: track 0.00 -> 45.6 mm, vias 0 -> 5
- net TIM8_CH1: track 0.00 -> 44.1 mm, vias 0 -> 2
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- added copper zone on B.Cu, net /halfHbridge4/GND_mech
- added copper zone on F.Cu, net /halfHbridge4/GND_mech
- added copper zone on In1.Cu, net /halfHbridge4/GND_mech
- added copper zone on In2.Cu, net /halfHbridge4/GND_mech
- added copper zone on B.Cu, net /halfHbridge4/out1
- added copper zone on F.Cu, net /halfHbridge4/out1
- added copper zone on In1.Cu, net /halfHbridge4/out1
- added copper zone on In2.Cu, net /halfHbridge4/out1
- added copper zone on B.Cu, net /halfHbridge5/GND_mech
- added copper zone on F.Cu, net /halfHbridge5/GND_mech
- added copper zone on In1.Cu, net /halfHbridge5/GND_mech
- added copper zone on In2.Cu, net /halfHbridge5/GND_mech
- added copper zone on B.Cu, net /halfHbridge5/out1
- added copper zone on F.Cu, net /halfHbridge5/out1
- added copper zone on In1.Cu, net /halfHbridge5/out1
- added copper zone on In2.Cu, net /halfHbridge5/out1
- added copper zone on B.Cu, net /halfHbridge6/GND_mech
- added copper zone on F.Cu, net /halfHbridge6/GND_mech
- added copper zone on In1.Cu, net /halfHbridge6/GND_mech
- added copper zone on In2.Cu, net /halfHbridge6/GND_mech
- added copper zone on B.Cu, net /halfHbridge6/out1
- added copper zone on F.Cu, net /halfHbridge6/out1
- added copper zone on In1.Cu, net /halfHbridge6/out1
- added copper zone on In2.Cu, net /halfHbridge6/out1
- added copper zone on B.Cu, net /halfHbridge7/GND_mech
- added copper zone on F.Cu, net /halfHbridge7/GND_mech
- added copper zone on In1.Cu, net /halfHbridge7/GND_mech
- added copper zone on In2.Cu, net /halfHbridge7/GND_mech
- added copper zone on B.Cu, net /halfHbridge7/out1
- added copper zone on F.Cu, net /halfHbridge7/out1
- added copper zone on In1.Cu, net /halfHbridge7/out1
- added copper zone on In2.Cu, net /halfHbridge7/out1
- added copper zone on B.Cu, net /halfHbridge8/GND_mech
- added copper zone on F.Cu, net /halfHbridge8/GND_mech
- added copper zone on In1.Cu, net /halfHbridge8/GND_mech
- added copper zone on In2.Cu, net /halfHbridge8/GND_mech
- added copper zone on B.Cu, net /halfHbridge8/out1
- added copper zone on F.Cu, net /halfHbridge8/out1
- added copper zone on In1.Cu, net /halfHbridge8/out1
- added copper zone on In2.Cu, net /halfHbridge8/out1
- added copper zone on B.Cu, net /halfHbridge9/GND_mech
- added copper zone on F.Cu, net /halfHbridge9/GND_mech
- added copper zone on In1.Cu, net /halfHbridge9/GND_mech
- added copper zone on In2.Cu, net /halfHbridge9/GND_mech
- added copper zone on B.Cu, net /halfHbridge9/out1
- added copper zone on F.Cu, net /halfHbridge9/out1
- added copper zone on In1.Cu, net /halfHbridge9/out1
- added copper zone on In2.Cu, net /halfHbridge9/out1
- added copper zone on B.Cu, net GND
- added copper zone on F.Cu, net GND
- added copper zone on In1.Cu, net GND
- added copper zone on In2.Cu, net GND
- added copper zone on B.Cu, net VCC
- added copper zone on F.Cu, net VCC
- added copper zone on In1.Cu, net VCC
- added copper zone on In2.Cu, net VCC
Other:
- copper layers 2 -> 4
- board text added: "+"
- board text added: "-"
- board text added: "10kΩ"
- board text added: "120Ω"
- board text added: "12V"
- board text added: "18V"
- board text added: "1kΩ"
- board text added: "2.4kΩ"
- board text added: "3.3V"
- board text added: "4.7kΩ"
- board text added: "5.0V"
- board text added: "5V"
- board text added: "660Ω"
- board text added: "A"
- board text added: "B"
- board text added: "Button"
- board text added: "C/Z"
- board text added: "CLK"
- board text added: "DIO"
- board text added: "G"
- board text added: "GND"
- board text added: "H"
- board text added: "L"
- board text added: "RST"
- board text added: "RX"
- board text added: "SCL"
- board text added: "SDA"
- board text added: "STM32G431CBU6"
- board text added: "TX"
