File: kicad/ESC_v2/ESC_v2.kicad_sch (KiCad schematic)
At the start: 63 parts, among them J1 Conn_01x05_Pin, J10 Conn_01x01_Pin, J11 Conn_01x01_Pin, J12 Conn_01x01_Pin, J13 Conn_01x03_Pin, J14 Conn_01x01_Pin, J15 Conn_01x01_Pin, J16 Conn_01x01_Pin, J2 Conn_01x05_Pin, J3 Conn_01x03_Pin, J4 Conn_01x03_Pin, J6 Conn_01x06_Pin, J7 Conn_01x02_Pin, J8 Conn_01x04_Pin, J9 Conn_01x02_Pin, U10 BD4104, U11 AMS1117-5.0, U12 ACS711xEXLT-15AB, U13 LM2937xMP, U19 STM32G431CBUx, U7 AMS1117-3.3, U8 ACS711xEXLT-15AB, U9 ACS711xEXLT-15AB

Commit message: add ESC_v3 final ver
Parts:
- removed C31: 470u, Capacitor_SMD:C_Elec_10x10.2, symbol Device:C
- removed J10, J11, J12, J14, J15, J16: Conn_01x01_Pin, TestPoint:TestPoint_Pad_3.0x3.0mm, symbol Connector:Conn_01x01_Pin
- removed J13: Conn_01x03_Pin, Connector_Molex:Molex_KK-254_AE-6410-03A_1x03_P2.54mm_Vertical, symbol Connector:Conn_01x03_Pin
- removed J3, J4: Conn_01x03_Pin, Connector_PinSocket_2.54mm:PinSocket_1x03_P2.54mm_Vertical, symbol Connector:Conn_01x03_Pin
- added C23, C39: 0.1u, Capacitor_SMD:C_0402_1005Metric, symbol Device:C
- added C40, C41, C42, C43, C44, C45, C46, C47, C48, C49: 22uF, Capacitor_SMD:C_0603_1608Metric, symbol Device:C
- added D2: 1N5819WS, Diode_SMD:D_SOD-323, symbol Diode:1N5819WS
- added J3: Conn_01x01_Pin, Connector_PinHeader_1.00mm:PinHeader_1x01_P1.00mm_Vertical, symbol Connector:Conn_01x01_Pin
- added J5: Conn_01x02_Pin, Connector_PinHeader_2.54mm:PinHeader_1x02_P2.54mm_Vertical, symbol Connector:Conn_01x02_Pin
- added NRST1, button1: SW_Push, jisaku:Aitendo_SW SMD 6x3.5, symbol Switch:SW_Push
- added R5, R6: 10k, Resistor_SMD:R_0402_1005Metric_Pad0.72x0.64mm_HandSolder, symbol Device:R
- added TP1, TP10, TP11, TP12, TP2, TP3, TP4, TP5, TP6, TP7, TP8, TP9: TestPoint, TestPoint:TestPoint_Pad_D1.0mm, symbol Connector:TestPoint
- C38: value 1u -> 0.1u
- D15, D16, D17: footprint LED_SMD:LED_0805_2012Metric -> LED_SMD:LED_0603_1608Metric
- J7: footprint Connector_JST:JST_XH_B2B-XH-AM_1x02_P2.50mm_Vertical -> Connector_JST:JST_XH_S2B-XH-A_1x02_P2.50mm_Horizontal
- R48, R49, R54: value 22k -> 68k
- R51: footprint Resistor_SMD:R_0402_1005Metric_Pad0.72x0.64mm_HandSolder -> Resistor_SMD:R_2010_5025Metric_Pad1.40x2.65mm_HandSolder
Connections:
- net +12V: no longer C29.1, U7.3 (VI)
- net +3.3V: now also R5.1, R6.2
- net +5V: now also C29.1, J1.1 (Pin_1), J2.1 (Pin_1), J6.1 (Pin_1), U7.3 (VI), D2.1 (K); no longer U11.2 (VO)
- net ADC2_IN14: now also U19.12 (PA4); no longer U19.24 (PB11)
- net ADC2_IN15: now also U19.13 (PA5); no longer U19.28 (PB15)
- net CAN_H: now also J7.2 (Pin_2), J5.2 (Pin_2); no longer J7.1 (Pin_1), R43.2
- net CAN_L: now also J7.1 (Pin_1); no longer J7.2 (Pin_2)
- net GND: now also J9.1 (Pin_1), C23.2, C39.2, C40.2, C41.2, C42.2, C43.2, C44.2, C45.2, C46.2, C47.2, C48.2, C49.2, J3.1 (Pin_1), NRST1.1, button1.1; no longer J9.2 (Pin_2), U19.11 (PA3), U19.13 (PA5), U19.19 (PB2)
- net OPAMP1_VINP: now also U19.11 (PA3); no longer U19.15 (PA7)
- net OPAMP2_VINP: now also U19.15 (PA7); no longer U19.27 (PB14)
- net RX: now also U19.24 (PB11); no longer U19.42 (PB4)
- net TIM1_CH1: now also TP1.1
- net TIM1_CH1N: now also TP2.1
- net TIM1_CH2: now also TP3.1
- net TIM1_CH2N: now also U19.27 (PB14), TP4.1; no longer U19.17 (PB0)
- net TIM1_CH3: now also TP5.1
- net TIM1_CH3N: now also U19.28 (PB15), TP6.1; no longer U19.18 (PB1)
- net TIM2_CH1: now also J2.2 (Pin_2); no longer J2.1 (Pin_1)
- net TIM3_CH1: now also J1.2 (Pin_2), U19.42 (PB4); no longer J1.1 (Pin_1), U19.14 (PA6)
- net TIM3_CH2: now also U19.43 (PB5); no longer U19.12 (PA4)
- net TIM8_CH1: now also TP11.1
- net TIM8_CH1N: now also TP12.1
- net TIM8_CH2: now also TP9.1
- net TIM8_CH2N: now also TP10.1
- net TIM8_CH3: now also TP7.1
- net TIM8_CH3N: now also U19.18 (PB1), TP8.1; no longer U19.43 (PB5)
- net TX: now also U19.22 (PB10); no longer U19.10 (PA2)
- net VCC: now also J9.2 (Pin_2), C40.1, C41.1, C42.1, C43.1, C44.1, C45.1, C46.1, C47.1, C48.1, C49.1; no longer J9.1 (Pin_1)
- net button: now reaches U19.29 (PC6)
- net button: now also C39.1, R5.2, button1.2
- net NRST: now reaches U19.7 (PG10)
- net NRST: now also C23.1, NRST1.2, R6.1
- net TIM2_ETR renamed TIM2_CH3
- net TIM2_CH3: now also U19.10 (PA2)
- net TIM3_ETR renamed TIM3_CH3
- net TIM3_CH3: now also U19.17 (PB0)
- net TIM4_CH1 renamed TIM4_CH2
- new net: D2.2 (A), U11.2 (VO)
- new net: J5.1 (Pin_1), R43.2
- new net OPAMP3_VINM0: U19.19 (PB2)
Other:
- removed sheet led_out
- removed sheet led_out1
- removed sheet led_out2
- removed sheet led_out3
- removed sheet led_out4
- removed sheet led_out5
- moved on the sheet: C16, C19, C20, C26, C3, C32, J7, J9, R43, U10
